Commit message: working version

File: urdf/robmobile.xacro (robot description, xacro)
@@ -11,5 +11,5 @@
   </inertial>
   <visual>
-    <origin rpy="0 0 1.570796" xyz="0.325 0 0.625"/> <!-- COM: CHECK : Update 0.625 -->
+    <origin rpy="0 0 0" xyz="0.325 0 0.625"/> <!-- COM: CHECK : Update 0.625 -->
     <geometry>
       <mesh filename="package://robmobile_description/meshes/base_link.stl" scale="0.001 0.001 0.001"/>
@@ -18,5 +18,5 @@
   </visual>
   <collision>
-    <origin rpy="0 0 1.570796" xyz="0.325 0 0.625"/>
+    <origin rpy="0 0 0" xyz="0.325 0 0.625"/>
     <geometry>
       <mesh filename="package://robmobile_description/meshes/base_link.stl" scale="0.001 0.001 0.001"/>
@@ -45,5 +45,5 @@
 </link>
 <joint name="l_wheel_joint" type="continuous">
-  <origin rpy="0 0 1.570796" xyz="-0.325 0 -0.105"/>
+  <origin rpy="0 0 0" xyz="-0.325 0 -0.105"/>
   <parent link="base_link"/>
   <child link="l_wheel"/>
@@ -57,5 +57,5 @@
   </inertial>
   <visual>
-    <origin rpy="0 0 0" xyz="-0.65 0 0.73"/>
+    <origin rpy="0 0 3.14159" xyz="-0.65 0 0.73"/>
     <geometry>
       <mesh filename="package://robmobile_description/meshes/wheel.stl" scale="0.001 0.001 0.001"/>
@@ -64,5 +64,5 @@
   </visual>
   <collision>
-    <origin rpy="0 0 0" xyz="-0.65 0 0.73"/>
+    <origin rpy="0 0 3.14159" xyz="-0.65 0 0.73"/>
     <geometry>
       <mesh filename="package://robmobile_description/meshes/wheel.stl" scale="0.001 0.001 0.001"/>
@@ -71,5 +71,5 @@
 </link>
 <joint name="r_wheel_joint" type="continuous">
-  <origin rpy="0 0 1.570796" xyz="0.325 0 -0.105"/>
+  <origin rpy="0 0 0" xyz="0.325 0 -0.105"/>
   <parent link="base_link"/>
   <child link="r_wheel"/>
@@ -97,5 +97,5 @@
 </link>
 <joint name="lf_swivel_joint" type="continuous">
-  <origin rpy="0 0 1.570796" xyz="-0.25 0.45 -0.03"/>
+  <origin rpy="0 0 0" xyz="-0.25 0.45 -0.03"/>
   <parent link="base_link"/>
   <child link="lf_swivel"/>
@@ -123,5 +123,5 @@
 </link>
 <joint name="rf_swivel_joint" type="continuous">
-  <origin rpy="0 0 1.570796" xyz="0.25 0.45 -0.03"/>
+  <origin rpy="0 0 0" xyz="0.25 0.45 -0.03"/>
   <parent link="base_link"/>
   <child link="rf_swivel"/>
@@ -149,8 +149,8 @@
 </link>
 <joint name="rb_swivel_joint" type="continuous">
-  <origin rpy="0 0 1.570796" xyz="0.25 -0.45 -0.03"/>
+  <origin rpy="0 0 0" xyz="0.25 -0.45 -0.03"/>
   <parent link="base_link"/>
   <child link="rb_swivel"/>
-  <axis xyz="0.0 0.0 1.0"/>
+  <axis xyz="0.0 -0.0 1.0"/>
 </joint>
 <link name="lb_swivel">
@@ -175,5 +175,5 @@
 </link>
 <joint name="lb_swivel_joint" type="continuous">
-  <origin rpy="0 0 1.570796" xyz="-0.25 -0.45 -0.03"/>
+  <origin rpy="0 0 0" xyz="-0.25 -0.45 -0.03"/>
   <parent link="base_link"/>
   <child link="lb_swivel"/>
@@ -204,5 +204,5 @@
   <parent link="rf_swivel"/>
   <child link="rf_caster_wheel"/>
-  <axis xyz="1.0 0.0 0.0"/>
+  <axis xyz="0.0 1.0 0.0"/>
 </joint>
 <link name="lf_caster_wheel">
@@ -230,5 +230,5 @@
   <parent link="lf_swivel"/>
   <child link="lf_caster_wheel"/>
-  <axis xyz="-1.0 0.0 0.0"/>
+  <axis xyz="0.0 1.0 0.0"/>
 </joint>
 <link name="rb_caster_wheel">
@@ -256,5 +256,5 @@
   <parent link="rb_swivel"/>
   <child link="rb_caster_wheel"/>
-  <axis xyz="1.0 0.0 0.0"/>
+  <axis xyz="0.0 1.0 0.0"/>
 </joint>
 <link name="lb_caster_wheel">
@@ -282,5 +282,5 @@
   <parent link="lb_swivel"/>
   <child link="lb_caster_wheel"/>
-  <axis xyz="-1.0 0.0 0.0"/>  <!-- IMP: Update -->
+  <axis xyz="0.0 1.0 0.0"/>  <!-- IMP: Update -->
   <dynamics damping="0"/>
 </joint>
@@ -306,8 +306,8 @@
 </link>
 <joint name="lidar" type="fixed"> <!-- Update -->
-  <origin rpy="0 0 3.141592" xyz="0.0 0.15 0.642"/>
+  <origin rpy="1.570796 0 -1.570796" xyz="0.0 0.15 0.642"/> <!-- 0 0 3.141592 -->
   <parent link="base_link"/>
   <child link="lidar_1"/>
-  <!--axis xyz="0.0 0.0 1.0"/-->
+  <!--axis xyz="0.0 0.0 1.0"/-->     <!-- comment this line too -->
 </joint>
 </robot>
